File: EAGLE/ESP-AC_LAR/placaESP-AC_LAR_01.brd (EAGLE design)
At the start: 42.5 x 44.5 mm, 12 parts, among them Q1 2N4416

Commit message: Peq. alteração
Parts:
- IR: value SFH482 -> (none)
- Q1: value 2N4416 -> 2N4401
Changed lines of the file:
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@@
 </autorouter>
 <elements>
-<element name="IR" library="led" package="SFH482" value="SFH482" x="36.45" y="7.93" rot="R270"/>
+<element name="IR" library="led" package="SFH482" value="" x="36.45" y="7.93" rot="R270"/>
 <element name="FTDI" library="con-lstb" package="MA06-1" value="" x="13.66" y="2.81">
 <attribute name="OC_NEWARK" value="unknown" x="13.66" y="2.81" size="1.778" layer="27" display="off"/>
@@
 </element>
 <element name="MDL1" library="ESP8266-ESP12E" package="ESP8266-ESP12E" value="" x="16.51" y="31.75" rot="R90"/>
-<element name="Q1" library="transistor-npn" package="TO92" value="2N4416" x="19.92" y="9.17" rot="R90"/>
+<element name="Q1" library="transistor-npn" package="TO92" value="2N4401" x="19.92" y="9.17" rot="R90"/>
 <element name="RESET" library="switch-omron" package="B3F-10XX" value="" x="36.95" y="27.4">
 <attribute name="OC_NEWARK" value="36M3542" x="36.95" y="27.4" size="1.778" layer="27" display="off"/>

Commit message: Meloria no botão de flash
Parts:
- added R6: 10k, rcl:0207/10
Connections:
- removed net N$7: FLASH.4, MDL1.12
- new net N$6: FLASH.3, FLASH.4, MDL1.12, R6.1
- net VCC: now also R6.2; no longer FLASH.3
Routing:
- net N$7: track 16.1 -> 0.00 mm
- added copper zone on layer 1, net GND
- added copper zone on layer 16, net GND
Changed lines of the file:
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@@
 <element name="R5" library="rcl" package="0207/10" value="100R" x="22.594" y="15.06"/>
 <element name="C1" library="rcl" package="C025-025X050" value="100n" x="33.5" y="18.922" rot="R90"/>
+<element name="R6" library="rcl" package="0207/10" value="10k" x="9" y="-11.5"/>
 </elements>
 <signals>
 <signal name="VCC">
 <contactref element="MDL1" pad="8"/>
-<contactref element="FLASH" pad="3"/>
 <contactref element="FTDI" pad="4"/>
 <contactref element="R2" pad="1"/>
@@
 <wire x1="35.6616" y1="22.4028" x2="35.6616" y2="34.5186" width="0.254" layer="16"/>
 <wire x1="33.6042" y1="20.3454" x2="35.6616" y2="22.4028" width="0.254" layer="16"/>
-<wire x1="40.005" y1="40.9194" x2="40.2012" y2="41.0906" width="0.254" layer="16"/>
 <wire x1="33.6042" y1="20.3454" x2="33.5" y2="20.192" width="0.254" layer="16"/>
 <wire x1="16.6878" y1="14.859" x2="9.8298" y2="8.001" width="0.254" layer="16"/>
 <wire x1="17.3736" y1="14.859" x2="16.6878" y2="14.859" width="0.254" layer="16"/>
 <wire x1="17.3736" y1="14.859" x2="17.514" y2="15.06" width="0.254" layer="16"/>
+<contactref element="R6" pad="2"/>
+<wire x1="14.08" y1="-11.5" x2="14.93" y2="2.81" width="0" layer="19" extent="1-1"/>
 </signal>
 <signal name="GND">
@@
 <wire x1="40.005" y1="36.3474" x2="40.2012" y2="36.5694" width="0.254" layer="16"/>
 <wire x1="40.005" y1="25.146" x2="40.2012" y2="25.1394" width="0.254" layer="16"/>
+<polygon width="0.254" layer="16">
+<vertex x="0" y="0"/>
+<vertex x="0" y="44.5"/>
+<vertex x="42.5" y="44.5"/>
+<vertex x="42.5" y="0"/>
+</polygon>
+<polygon width="0.254" layer="1">
+<vertex x="0" y="0"/>
+<vertex x="42.5" y="0"/>
+<vertex x="42.5" y="44.5"/>
+<vertex x="0" y="44.5"/>
+</polygon>
 </signal>
 <signal name="CTS">
@@
 <wire x1="4.1148" y1="18.5166" x2="3.9" y2="18.708" width="0.254" layer="16"/>
 </signal>
-<signal name="N$7">
-<contactref element="MDL1" pad="12"/>
-<contactref element="FLASH" pad="4"/>
-<wire x1="19.6596" y1="41.3766" x2="18.7452" y2="40.4622" width="0.254" layer="1"/>
-<wire x1="19.6596" y1="41.6052" x2="19.6596" y2="41.3766" width="0.254" layer="1"/>
-<wire x1="19.8882" y1="41.8338" x2="19.6596" y2="41.6052" width="0.254" layer="1"/>
-<wire x1="32.9184" y1="41.8338" x2="19.8882" y2="41.8338" width="0.254" layer="1"/>
-<wire x1="33.6042" y1="41.148" x2="32.9184" y2="41.8338" width="0.254" layer="1"/>
-<wire x1="18.7452" y1="40.4622" x2="18.67" y2="40.33" width="0.254" layer="1"/>
-<wire x1="33.6042" y1="41.148" x2="33.6988" y2="41.0906" width="0.254" layer="1"/>
-</signal>
 <signal name="RXI">
 <contactref element="MDL1" pad="16"/>
@@
 <wire x1="12.1158" y1="18.5166" x2="12.11" y2="18.63" width="0.254" layer="1"/>
 </signal>
+<signal name="N$6">
+<contactref element="FLASH" pad="3"/>
+<contactref element="FLASH" pad="4"/>
+<contactref element="MDL1" pad="12"/>
+<contactref element="R6" pad="1"/>
+<wire x1="33.6988" y1="41.0906" x2="40.2012" y2="41.0906" width="0" layer="19" extent="1-1"/>
+<wire x1="18.67" y1="40.33" x2="33.6988" y2="41.0906" width="0" layer="19" extent="1-1"/>
+<wire x1="3.92" y1="-11.5" x2="18.67" y2="40.33" width="0" layer="19" extent="1-1"/>
+</signal>
 </signals>
